Commit message: Add functional Blender centrifuge to the laboratory
Add articulated rotor and lid assets, open sample holders, contact-verified loading, balanced timed MuJoCo cycles, browser controls and protected API routes. Include the instrument in the portable CRAM world and prevent conflicting robot operations.

Validated physical loading, timed rotation, braking, unloading and reseating; existing PR2 mixing, transfer, weighing and server regressions; authenticated local and deployed full-cycle checks.

File: src/cramera/resources/precision_lab/environment.urdf (robot description, URDF)
Before this commit: robot precision_laboratory, 4 links, 3 joints
Links:
- added link laboratory_balance; collision box size=0.0045 0.0042128799 0.04; collision box size=0.0045 0.0042128799 0.04
- added link laboratory_centrifuge_base; collision box size=0.013 0.039495749 0.181; collision box size=0.013 0.039495749 0.181
- added link laboratory_centrifuge_lid, mass 0.55; collision box size=0.3 0.3 0.014; visual mesh filename=assets/centrifuge_lid.glb
- added link laboratory_centrifuge_rotor, mass 0.4; collision box size=0.0045 0.0063651958 0.115; collision box size=0.0045 0.0063651958 0.115
Joints:
- added joint laboratory_balance_joint: type fixed, parent laboratory_root, child laboratory_balance, origin xyz=0.65 0.21 0.968 rpy=0 0 0
- added joint laboratory_centrifuge_base_joint: type fixed, parent laboratory_root, child laboratory_centrifuge_base, origin xyz=-0.53 -0.07 0.9 rpy=0 0 0
- added joint laboratory_centrifuge_lid_joint: type revolute, parent laboratory_centrifuge_base, child laboratory_centrifuge_lid, origin xyz=0 0.155 0.223 rpy=0 0 0, axis -1 0 0, limit lower=0 upper=1.85 effort=8 velocity=1
- added joint laboratory_centrifuge_rotor_joint: type continuous, parent laboratory_centrifuge_base, child laboratory_centrifuge_rotor, origin xyz=0 0 0.052 rpy=0 0 0, axis 0 0 1

Commit message: Add functional pipetting station and PR2 dosing demo

File: src/cramera/resources/precision_lab/environment.urdf (robot description, URDF)
Before this commit: robot precision_laboratory, 8 links, 7 joints
Links:
- added link laboratory_pipetting_station; collision box size=0.0016 0.0016 0.027; collision box size=0.0016 0.0016 0.027
Joints:
- added joint laboratory_pipetting_station_joint: type fixed, parent laboratory_root, child laboratory_pipetting_station, origin xyz=-0.1 0 0.9 rpy=0 0 0

Commit message: Add articulated sample refrigerator with contact-guided storage

File: src/cramera/resources/precision_lab/environment.urdf (robot description, URDF)
Before this commit: robot precision_laboratory, 9 links, 8 joints
Links:
- added link laboratory_refrigerator_base; collision box size=0.007 0.0073597576 0.04; collision box size=0.007 0.0073597576 0.04
- added link laboratory_refrigerator_door, mass 3.0; collision box size=0.036 0.032 0.58; collision box size=0.036 0.032 0.58
Joints:
- added joint laboratory_refrigerator_base_joint: type fixed, parent laboratory_root, child laboratory_refrigerator_base, origin xyz=-1.23 0 0 rpy=0 0 0
- added joint laboratory_refrigerator_door_joint: type revolute, parent laboratory_refrigerator_base, child laboratory_refrigerator_door, origin xyz=-0.25 -0.31 0.43 rpy=0 0 0, axis 0 0 -1, limit lower=0 upper=1.75 effort=15 velocity=1
