Commit message: Operate laboratory covers through PR2 handle contacts

File: src/cramera/resources/laboratory_devices/centrifuge/model.urdf (robot description, URDF)
Before this commit: robot centrifuge, 3 links, 2 joints
Links:
- link laboratory_centrifuge_lid: geometry collision box size=0.014 0.016 0.086; collision box size=0.014 0.016 0.086
Joints:
- joint laboratory_centrifuge_lid_joint: limit lower=0 upper=1.85 effort=8 velocity=1 -> lower=0 upper=1.35 effort=8 velocity=1

File: src/cramera/resources/laboratory_devices/refrigerator/model.urdf (robot description, URDF)
Before this commit: robot refrigerator, 2 links, 1 joints
Links:
- link laboratory_refrigerator_door: geometry collision box size=0.016 0.035 0.016; collision box size=0.016 0.035 0.016

File: src/cramera/resources/precision_lab/environment.urdf (robot description, URDF)
Before this commit: robot precision_laboratory, 11 links, 10 joints
Links:
- link laboratory_centrifuge_lid: geometry collision box size=0.014 0.016 0.086; collision box size=0.014 0.016 0.086
- link laboratory_refrigerator_door: geometry collision box size=0.016 0.035 0.016; collision box size=0.016 0.035 0.016
Joints:
- joint laboratory_centrifuge_base_joint: origin xyz=-0.53 -0.07 0.9 rpy=0 0 0 -> xyz=-0.53 -0.18 0.9 rpy=0 0 0
- joint laboratory_centrifuge_lid_joint: limit lower=0 upper=1.85 effort=8 velocity=1 -> lower=0 upper=1.35 effort=8 velocity=1

Commit message: Expose named laboratory handle frames in CRAM and the viewer

File: src/cramera/resources/laboratory_devices/centrifuge/model.urdf (robot description, URDF)
Before this commit: robot centrifuge, 3 links, 2 joints
Links:
- added link laboratory_centrifuge_lid_handle
Joints:
- added joint laboratory_centrifuge_lid_handle_joint: type fixed, parent laboratory_centrifuge_lid, child laboratory_centrifuge_lid_handle, origin xyz=0 -0.21 0.09 rpy=0 0 0

File: src/cramera/resources/laboratory_devices/refrigerator/model.urdf (robot description, URDF)
Before this commit: robot refrigerator, 2 links, 1 joints
Links:
- added link laboratory_refrigerator_door_handle
Joints:
- added joint laboratory_refrigerator_door_handle_joint: type fixed, parent laboratory_refrigerator_door, child laboratory_refrigerator_door_handle, origin xyz=0.482 -0.044 0 rpy=0 0 0

File: src/cramera/resources/precision_lab/environment.urdf (robot description, URDF)
Before this commit: robot precision_laboratory, 11 links, 10 joints
Links:
- added link laboratory_cabinet_lower_handle
- added link laboratory_cabinet_middle_handle
- added link laboratory_cabinet_right_handle
- added link laboratory_centrifuge_lid_handle
- added link laboratory_drawer_handle
- added link laboratory_refrigerator_door_handle
Joints:
- added joint laboratory_cabinet_lower_handle_joint: type fixed, parent laboratory_room, child laboratory_cabinet_lower_handle, origin xyz=-0.52 -0.346 0.546 rpy=0 0 0
- added joint laboratory_cabinet_middle_handle_joint: type fixed, parent laboratory_room, child laboratory_cabinet_middle_handle, origin xyz=0.005 -0.346 0.744 rpy=0 0 0
- added joint laboratory_cabinet_right_handle_joint: type fixed, parent laboratory_room, child laboratory_cabinet_right_handle, origin xyz=0.523 -0.346 0.744 rpy=0 0 0
- added joint laboratory_centrifuge_lid_handle_joint: type fixed, parent laboratory_centrifuge_lid, child laboratory_centrifuge_lid_handle, origin xyz=0 -0.21 0.09 rpy=0 0 0
- added joint laboratory_drawer_handle_joint: type fixed, parent laboratory_drawer, child laboratory_drawer_handle, origin xyz=0 -0.336 0.015 rpy=0 0 0
- added joint laboratory_refrigerator_door_handle_joint: type fixed, parent laboratory_refrigerator_door, child laboratory_refrigerator_door_handle, origin xyz=0.482 -0.044 0 rpy=0 0 0
