Commit message: Retrieve the loaded sample rack before the laboratory workflow
Start the native Coraplex recipe by opening the drawer, carrying the rack of
four empty samples to the bench, and closing the drawer. Model the carrier
and samples as separate contact-driven bodies, include the carried assembly
in base clearance checks, and preserve measured rack and handle poses in the
semantic world, live viewer and recordings.

Update the Blender authoring and portable rack resources with a carry handle
and flared sample guides. Require complete drawer withdrawal before torso
recovery and keep interpolated joint commands within their authored limits.

File: src/cramera/resources/laboratory_devices/tube_rack/model.urdf (robot description, URDF)
Before this commit: robot tube_rack, 1 links, 0 joints
Links:
- added link laboratory_rack_handle
- link laboratory_rack: mass None -> 0.18; geometry collision box size=0.0023717082 0.0075025774 0.0063245553; collision box size=0.0023717082 0.0075025774 0.0063245553
Joints:
- added joint laboratory_rack_handle_joint: type fixed, parent laboratory_rack, child laboratory_rack_handle, origin xyz=0 -0.125 0.055 rpy=0 0 0

File: src/cramera/resources/precision_lab/environment.urdf (robot description, URDF)
Before this commit: robot precision_laboratory, 17 links, 16 joints
Links:
- added link laboratory_rack_handle
- link laboratory_drawer: geometry collision box size=0.012 0.025 0.014; collision box size=0.012 0.025 0.014
- link laboratory_rack: mass None -> 0.18; geometry collision box size=0.0023717082 0.0075025774 0.0063245553; collision box size=0.0023717082 0.0075025774 0.0063245553
Joints:
- added joint laboratory_rack_handle_joint: type fixed, parent laboratory_rack, child laboratory_rack_handle, origin xyz=0 -0.125 0.055 rpy=0 0 0
- joint laboratory_rack_joint: type fixed -> floating
