Commit message: Add MuJoCo workshop contacts and tool-driven screw insertion

File: src/cramera/resources/aicor_workshop/environment.urdf (robot description, URDF)
Before this commit: robot aicor_workshop, 10 links, 9 joints
Links:
- removed link workshop_assembly
- removed link workshop_socket
- link workshop_drawer_1: geometry collision box size=0.009 0.56 0.14; collision box size=0.009 0.56 0.14
- link workshop_drawer_1_handle: geometry collision box size=0.016 0.028 0.018; collision box size=0.016 0.028 0.018
- link workshop_drawer_2: geometry collision box size=0.009 0.56 0.14; collision box size=0.009 0.56 0.14
- link workshop_drawer_2_handle: geometry collision box size=0.016 0.028 0.018; collision box size=0.016 0.028 0.018
- link workshop_drawer_3: geometry collision box size=0.009 0.56 0.14; collision box size=0.009 0.56 0.14
- link workshop_drawer_3_handle: geometry collision box size=0.016 0.028 0.018; collision box size=0.016 0.028 0.018
- link workshop_environment: geometry collision box size=0.004 0.5 0.018; collision box size=0.004 0.5 0.018
Joints:
- removed joint workshop_assembly_joint
- removed joint workshop_socket_joint

File: src/cramera/resources/aicor_workshop/screw_1.urdf (robot description, URDF)
Before this commit: robot screw_1, 1 links, 0 joints
Links:
- link screw_1: geometry collision box size=0.0055166605 0.006 0.006; collision box size=0.0055166605 0.006 0.006

File: src/cramera/resources/aicor_workshop/screw_2.urdf (robot description, URDF)
Before this commit: robot screw_2, 1 links, 0 joints
Links:
- link screw_2: geometry collision box size=0.0055166605 0.006 0.006; collision box size=0.0055166605 0.006 0.006

File: src/cramera/resources/aicor_workshop/screw_3.urdf (robot description, URDF)
Before this commit: robot screw_3, 1 links, 0 joints
Links:
- link screw_3: geometry collision box size=0.0055166605 0.006 0.006; collision box size=0.0055166605 0.006 0.006

File: src/cramera/resources/aicor_workshop/screw_4.urdf (robot description, URDF)
Before this commit: robot screw_4, 1 links, 0 joints
Links:
- link screw_4: geometry collision box size=0.0055166605 0.006 0.006; collision box size=0.0055166605 0.006 0.006

File: src/cramera/resources/aicor_workshop/screw_5.urdf (robot description, URDF)
Before this commit: robot screw_5, 1 links, 0 joints
Links:
- link screw_5: geometry collision box size=0.0055166605 0.006 0.006; collision box size=0.0055166605 0.006 0.006

Commit message: workbench and inno

File: src/cramera/resources/aicor_workshop/environment.urdf (robot description, URDF)
Before this commit: robot aicor_workshop, 8 links, 7 joints
Links:
- link workshop_environment: geometry collision box size=0.004 0.5 0.018; collision box size=0.004 0.5 0.018

File: src/cramera/resources/aicor_workshop/nail_box.urdf (robot description, URDF)
Before this commit: robot nail_box, 1 links, 0 joints
Links:
- added link nail_box_handle; collision box size=0.012 0.042 0.018; collision box size=0.012 0.042 0.018
Joints:
- added joint nail_box_handle_joint: type fixed, parent nail_box, child nail_box_handle, origin xyz=0 -0.204 0.055 rpy=0 0 0

File: src/cramera/resources/aicor_workshop/screw_box.urdf (robot description, URDF)
Before this commit: robot screw_box, 1 links, 0 joints
Links:
- added link screw_box_handle; collision box size=0.012 0.042 0.018; collision box size=0.012 0.042 0.018
Joints:
- added joint screw_box_handle_joint: type fixed, parent screw_box, child screw_box_handle, origin xyz=0 -0.204 0.055 rpy=0 0 0

File: src/cramera/resources/aicor_workshop/workshop_assembly.urdf (robot description, URDF)
Before this commit: robot workshop_assembly, 2 links, 1 joints
Links:
- link workshop_assembly: geometry collision box size=0.02 0.2 0.004; collision box size=0.02 0.2 0.004
