Commit message: Add the Designators layout: roles, designator tree and EQL resolution
?layout=designators shows the 3D scene beside three panes bound to the
top-level action at the playback frame: the SDT entities filling a role
in it (row <-> body selection), the action designator tree with role
slots and phases, and how each role was filled, by an entity query whose
answer is the same entity, from the plan context, or by the plan's code.
Answers are marked RECORDED or LIVE; the queries are EQL over the twin's
working memory, not KnowRob.

The bridge records each plan node's roles (FIELD_ROLES in names.py) and
stamps each query step with its frame, plan node and answer entities.
The PR2 workflow finds its vessels and handles by entity queries, and
aicor_medical_lab_pr2_workflow is re-recorded with its query steps,
including the refrigerator storage and centrifuge loading.

Co-Authored-By: Claude Opus 5.5 <noreply@anthropic.com>

File: demo/standard_scenes/aicor_medical_lab_pr2_workflow/environment.urdf (robot description, URDF)
Before this commit: robot environment, 21 links, 20 joints
Links:
- removed link 80dffb99-697d-4a08-bc45-75e67fb4e504/odom
- added link c83002c0-7c8c-45db-82c9-11bb0ee5c35a/odom
- link laboratory_centrifuge_base: geometry collision box size=0.013 0.039496 0.181; collision box size=0.013 0.039496 0.181
- link laboratory_centrifuge_lid: geometry collision box size=0.014 0.016 0.086; collision box size=0.014 0.016 0.086
- link laboratory_centrifuge_rotor: geometry collision box size=0.0045 0.006365 0.115; collision box size=0.0045 0.006365 0.115
- link laboratory_drawer: geometry collision box size=0.012 0.025 0.014; collision box size=0.012 0.025 0.014
- link laboratory_pipetting_station: geometry collision box size=0.0016 0.0016 0.027; collision box size=0.0016 0.0016 0.027
- link laboratory_refrigerator_base: geometry collision box size=0.007 0.00736 0.04; collision box size=0.007 0.00736 0.04
- link laboratory_refrigerator_door: geometry collision box size=0.016 0.035 0.016; collision box size=0.016 0.035 0.016
- link laboratory_room: geometry collision box size=0.04 0.04 0.86; collision box size=0.04 0.04 0.86
Joints:
- removed joint 80dffb99-697d-4a08-bc45-75e67fb4e504/map_T_odom
- added joint c83002c0-7c8c-45db-82c9-11bb0ee5c35a/map_T_odom: type fixed, parent map, child c83002c0-7c8c-45db-82c9-11bb0ee5c35a/odom, origin xyz=0.0 0.0 0.0 rpy=0.0 0.0 0.0

File: demo/standard_scenes/aicor_medical_lab_pr2_workflow/pr2.urdf (robot description, URDF)
Before this commit: robot pr2, 105 links, 104 joints
Links:
- link pr2/base_link: geometry collision mesh filename=meshes/recording/base_v0-7c37a8f0/base_L.stl scale=1.0 1.0 1.0; visual mesh filename=meshes/recording/base_v0-7c37a8f0/base.dae scale=1.0 1.0 1.0
- link pr2/bl_caster_l_wheel_link: geometry collision cylinder length=0.034 radius=0.074792; visual mesh filename=meshes/recording/base_v0-7c37a8f0/wheel.dae scale=1.0 1.0 1.0
- link pr2/bl_caster_r_wheel_link: geometry collision cylinder length=0.034 radius=0.074792; visual mesh filename=meshes/recording/base_v0-7c37a8f0/wheel.dae scale=1.0 1.0 1.0
- link pr2/bl_caster_rotation_link: geometry collision mesh filename=meshes/recording/base_v0-7c37a8f0/caster_L.stl scale=1.0 1.0 1.0; visual mesh filename=meshes/recording/base_v0-7c37a8f0/caster.stl scale=1.0 1.0 1.0
- link pr2/br_caster_l_wheel_link: geometry collision cylinder length=0.034 radius=0.074792; visual mesh filename=meshes/recording/base_v0-7c37a8f0/wheel.dae scale=1.0 1.0 1.0
- link pr2/br_caster_r_wheel_link: geometry collision cylinder length=0.034 radius=0.074792; visual mesh filename=meshes/recording/base_v0-7c37a8f0/wheel.dae scale=1.0 1.0 1.0
- link pr2/br_caster_rotation_link: geometry collision mesh filename=meshes/recording/base_v0-7c37a8f0/caster_L.stl scale=1.0 1.0 1.0; visual mesh filename=meshes/recording/base_v0-7c37a8f0/caster.stl scale=1.0 1.0 1.0
- link pr2/fl_caster_l_wheel_link: geometry collision cylinder length=0.034 radius=0.074792; visual mesh filename=meshes/recording/base_v0-7c37a8f0/wheel.dae scale=1.0 1.0 1.0
- link pr2/fl_caster_r_wheel_link: geometry collision cylinder length=0.034 radius=0.074792; visual mesh filename=meshes/recording/base_v0-7c37a8f0/wheel.dae scale=1.0 1.0 1.0
- link pr2/fl_caster_rotation_link: geometry collision mesh filename=meshes/recording/base_v0-7c37a8f0/caster_L.stl scale=1.0 1.0 1.0; visual mesh filename=meshes/recording/base_v0-7c37a8f0/caster.stl scale=1.0 1.0 1.0
- link pr2/fr_caster_l_wheel_link: geometry collision cylinder length=0.034 radius=0.074792; visual mesh filename=meshes/recording/base_v0-7c37a8f0/wheel.dae scale=1.0 1.0 1.0
- link pr2/fr_caster_r_wheel_link: geometry collision cylinder length=0.034 radius=0.074792; visual mesh filename=meshes/recording/base_v0-7c37a8f0/wheel.dae scale=1.0 1.0 1.0
- link pr2/fr_caster_rotation_link: geometry collision mesh filename=meshes/recording/base_v0-7c37a8f0/caster_L.stl scale=1.0 1.0 1.0; visual mesh filename=meshes/recording/base_v0-7c37a8f0/caster.stl scale=1.0 1.0 1.0
- link pr2/head_mount_kinect2_link: geometry collision box size=0.25 0.117597 0.050301; visual mesh filename=meshes/recording/sensors-07a920b9/microsoft_kinect2.dae scale=1.0 1.0 1.0
- link pr2/head_mount_link: geometry collision box size=0.106 0.2957 0.1552; visual mesh filename=meshes/recording/kinect_prosilica_v0-dc4c08c9/115x100_swept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 scale=0.001 0.001 0.001
- link pr2/head_pan_link: geometry collision mesh filename=meshes/recording/head_v0-5fb2c976/head_pan_L.stl scale=1.0 1.0 1.0; visual mesh filename=meshes/recording/head_v0-5fb2c976/head_pan.dae scale=1.0 1.0 1.0
- link pr2/head_tilt_link: geometry collision mesh filename=meshes/recording/head_v0-5fb2c976/head_tilt_L.stl scale=1.0 1.0 1.0; visual mesh filename=meshes/recording/head_v0-5fb2c976/head_tilt.dae scale=1.0 1.0 1.0
- link pr2/l_elbow_flex_link: geometry collision mesh filename=meshes/recording/upper_arm_v0-611c0460/elbow_flex.stl scale=1.0 1.0 1.0; visual mesh filename=meshes/recording/upper_arm_v0-611c0460/elbow_flex.dae scale=1.0 1.0 1.0
- link pr2/l_forearm_link: geometry collision mesh filename=meshes/recording/forearm_v0-f1752220/forearm.stl scale=1.0 1.0 1.0; visual mesh filename=meshes/recording/forearm_v0-f1752220/forearm.dae scale=1.0 1.0 1.0
- link pr2/l_forearm_roll_link: geometry collision mesh filename=meshes/recording/upper_arm_v0-611c0460/forearm_roll_L.stl scale=1.0 1.0 1.0; visual mesh filename=meshes/recording/upper_arm_v0-611c0460/forearm_roll.stl scale=1.0 1.0 1.0
- link pr2/l_gripper_l_finger_link: geometry collision mesh filename=meshes/recording/gripper_v0-bb7a33e2/l_finger.stl scale=1.0 1.0 1.0; visual mesh filename=meshes/recording/gripper_v0-bb7a33e2/l_finger.dae scale=1.0 1.0 1.0
- link pr2/l_gripper_l_finger_tip_link: geometry collision mesh filename=meshes/recording/gripper_v0-bb7a33e2/l_finger_tip.stl scale=1.0 1.0 1.0; visual mesh filename=meshes/recording/gripper_v0-bb7a33e2/l_finger_tip.dae scale=1.0 1.0 1.0
- link pr2/l_gripper_palm_link: geometry collision mesh filename=meshes/recording/gripper_v0-bb7a33e2/gripper_palm.stl scale=1.0 1.0 1.0; visual mesh filename=meshes/recording/gripper_v0-bb7a33e2/gripper_palm.dae scale=1.0 1.0 1.0
- link pr2/l_gripper_r_finger_link: geometry collision mesh filename=meshes/recording/gripper_v0-bb7a33e2/l_finger.stl scale=1.0 1.0 1.0; visual mesh filename=meshes/recording/gripper_v0-bb7a33e2/l_finger.dae scale=1.0 1.0 1.0
- link pr2/l_gripper_r_finger_tip_link: geometry collision mesh filename=meshes/recording/gripper_v0-bb7a33e2/l_finger_tip.stl scale=1.0 1.0 1.0; visual mesh filename=meshes/recording/gripper_v0-bb7a33e2/l_finger_tip.dae scale=1.0 1.0 1.0
- link pr2/l_shoulder_lift_link: geometry collision mesh filename=meshes/recording/shoulder_v0-4e52c6f3/shoulder_lift.stl scale=1.0 1.0 1.0; visual mesh filename=meshes/recording/shoulder_v0-4e52c6f3/shoulder_lift.dae scale=1.0 1.0 1.0
- link pr2/l_shoulder_pan_link: geometry collision mesh filename=meshes/recording/shoulder_v0-4e52c6f3/shoulder_pan.stl scale=1.0 1.0 1.0; visual mesh filename=meshes/recording/shoulder_v0-4e52c6f3/shoulder_pan.dae scale=1.0 1.0 1.0
- link pr2/l_torso_lift_side_item_profile_link: geometry collision box size=0.04 0.41 0.04; visual mesh filename=meshes/recording/cableguide-bc7839b7/item_Profil_8_40x40_le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 scale=1.0 1.0 1.0
- link pr2/l_upper_arm_link: geometry collision mesh filename=meshes/recording/upper_arm_v0-611c0460/upper_arm.stl scale=1.0 1.0 1.0; visual mesh filename=meshes/recording/upper_arm_v0-611c0460/upper_arm.dae scale=1.0 1.0 1.0
- link pr2/l_upper_arm_roll_link: geometry collision mesh filename=meshes/recording/shoulder_v0-4e52c6f3/upper_arm_roll_L.stl scale=1.0 1.0 1.0; visual mesh filename=meshes/recording/shoulder_v0-4e52c6f3/upper_arm_roll.stl scale=1.0 1.0 1.0
- link pr2/l_wrist_flex_link: geometry collision mesh filename=meshes/recording/forearm_v0-f1752220/wrist_flex.stl scale=1.0 1.0 1.0; visual mesh filename=meshes/recording/forearm_v0-f1752220/wrist_flex.dae scale=1.0 1.0 1.0
- link pr2/l_wrist_roll_link: geometry collision mesh filename=meshes/recording/forearm_v0-f1752220/wrist_roll_L.stl scale=1.0 1.0 1.0; visual mesh filename=meshes/recording/forearm_v0-f1752220/wrist_roll.stl scale=1.0 1.0 1.0
- link pr2/laser_tilt_mount_link: geometry collision mesh filename=meshes/recording/tilting_laser_v0-31feeb11/tilting_hokuyo_L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 scale=1.0 1.0 1.0; visual mesh filename=meshes/recording/tilting_laser_v0-31feeb11/tilting_hokuyo.d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 scale=1.0 1.0 1.0
- link pr2/m_torso_lift_side_item_profile_link: geometry collision box size=0.04 0.42 0.04; visual mesh filename=meshes/recording/cableguide-bc7839b7/item_Profil_8_40x40_le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 scale=1.0 1.0 1.0
- link pr2/r_elbow_flex_link: geometry collision mesh filename=meshes/recording/upper_arm_v0-611c0460/elbow_flex.stl scale=1.0 1.0 1.0; visual mesh filename=meshes/recording/upper_arm_v0-611c0460/elbow_flex.dae scale=1.0 1.0 1.0
- link pr2/r_forearm_link: geometry collision mesh filename=meshes/recording/forearm_v0-f1752220/forearm.stl scale=1.0 1.0 1.0; visual mesh filename=meshes/recording/forearm_v0-f1752220/forearm.dae scale=1.0 1.0 1.0
- link pr2/r_forearm_roll_link: geometry collision mesh filename=meshes/recording/upper_arm_v0-611c0460/forearm_roll_L.stl scale=1.0 1.0 1.0; visual mesh filename=meshes/recording/upper_arm_v0-611c0460/forearm_roll.stl scale=1.0 1.0 1.0
- link pr2/r_gripper_l_finger_link: geometry collision mesh filename=meshes/recording/gripper_v0-bb7a33e2/l_finger.stl scale=1.0 1.0 1.0; visual mesh filename=meshes/recording/gripper_v0-bb7a33e2/l_finger.dae scale=1.0 1.0 1.0
- link pr2/r_gripper_l_finger_tip_link: geometry collision mesh filename=meshes/recording/gripper_v0-bb7a33e2/l_finger_tip.stl scale=1.0 1.0 1.0; visual mesh filename=meshes/recording/gripper_v0-bb7a33e2/l_finger_tip.dae scale=1.0 1.0 1.0
- link pr2/r_gripper_palm_link: geometry collision mesh filename=meshes/recording/gripper_v0-bb7a33e2/gripper_palm.stl scale=1.0 1.0 1.0; visual mesh filename=meshes/recording/gripper_v0-bb7a33e2/gripper_palm.dae scale=1.0 1.0 1.0
- link pr2/r_gripper_r_finger_link: geometry collision mesh filename=meshes/recording/gripper_v0-bb7a33e2/l_finger.stl scale=1.0 1.0 1.0; visual mesh filename=meshes/recording/gripper_v0-bb7a33e2/l_finger.dae scale=1.0 1.0 1.0
- link pr2/r_gripper_r_finger_tip_link: geometry collision mesh filename=meshes/recording/gripper_v0-bb7a33e2/l_finger_tip.stl scale=1.0 1.0 1.0; visual mesh filename=meshes/recording/gripper_v0-bb7a33e2/l_finger_tip.dae scale=1.0 1.0 1.0
- link pr2/r_shoulder_lift_link: geometry collision mesh filename=meshes/recording/shoulder_v0-4e52c6f3/shoulder_lift.stl scale=1.0 1.0 1.0; visual mesh filename=meshes/recording/shoulder_v0-4e52c6f3/shoulder_lift.dae scale=1.0 1.0 1.0
- link pr2/r_shoulder_pan_link: geometry collision mesh filename=meshes/recording/shoulder_v0-4e52c6f3/shoulder_pan.stl scale=1.0 1.0 1.0; visual mesh filename=meshes/recording/shoulder_v0-4e52c6f3/shoulder_pan.dae scale=1.0 1.0 1.0
- link pr2/r_torso_lift_side_item_profile_link: geometry collision box size=0.04 0.41 0.04; visual mesh filename=meshes/recording/cableguide-bc7839b7/item_Profil_8_40x40_le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 scale=1.0 1.0 1.0
- link pr2/r_upper_arm_link: geometry collision mesh filename=meshes/recording/upper_arm_v0-611c0460/upper_arm.stl scale=1.0 1.0 1.0; visual mesh filename=meshes/recording/upper_arm_v0-611c0460/upper_arm.dae scale=1.0 1.0 1.0
- link pr2/r_upper_arm_roll_link: geometry collision mesh filename=meshes/recording/shoulder_v0-4e52c6f3/upper_arm_roll_L.stl scale=1.0 1.0 1.0; visual mesh filename=meshes/recording/shoulder_v0-4e52c6f3/upper_arm_roll.stl scale=1.0 1.0 1.0
- link pr2/r_wrist_flex_link: geometry collision mesh filename=meshes/recording/forearm_v0-f1752220/wrist_flex.stl scale=1.0 1.0 1.0; visual mesh filename=meshes/recording/forearm_v0-f1752220/wrist_flex.dae scale=1.0 1.0 1.0
- link pr2/r_wrist_roll_link: geometry collision mesh filename=meshes/recording/forearm_v0-f1752220/wrist_roll_L.stl scale=1.0 1.0 1.0; visual mesh filename=meshes/recording/forearm_v0-f1752220/wrist_roll.stl scale=1.0 1.0 1.0
- link pr2/t_torso_lift_side_item_profile_link: geometry collision box size=0.04 1.0 0.04; visual mesh filename=meshes/recording/cableguide-bc7839b7/item_Profil_8_40x40_le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 scale=1.0 1.0 1.0
- link pr2/torso_lift_link: geometry collision mesh filename=meshes/recording/torso_v0-783fb20d/torso_lift_L.stl scale=1.0 1.0 1.0; visual mesh filename=meshes/recording/torso_v0-783fb20d/torso_lift.dae scale=1.0 1.0 1.0
Joints:
- joint pr2/head_mount_kinect_rgb_optical_frame_joint: origin xyz=0.0 0.0 0.0 rpy=-1.570796 0.0 -1.570796 -> xyz=-0.0 -0.0 0.0 rpy=-1.570796 0.0 -1.570796
- joint pr2/imu_joint: origin xyz=-0.02977 -0.1497 0.164 rpy=3.141593 -0.0 3.141593 -> xyz=-0.02977 -0.1497 0.164 rpy=-3.141593 -0.0 -3.141593
- joint pr2/l_force_torque_adapter_joint: origin xyz=0.0356 0.0 0.0 rpy=0.0 -1.570796 0.0 -> xyz=0.0356 -0.0 0.0 rpy=0.0 -1.570796 0.0
- joint pr2/l_forearm_cam_optical_frame_joint: origin xyz=0.0 0.0 0.0 rpy=-1.570796 0.0 -1.570796 -> xyz=-0.0 0.0 0.0 rpy=-1.570796 0.0 -1.570796
- joint pr2/l_gripper_palm_joint: origin xyz=0.0 0.0 0.0 rpy=1.22173 1.570796 0.0 -> xyz=0.0 -0.0 0.0 rpy=1.22173 1.570796 0.0
- joint pr2/laser_tilt_joint: origin xyz=0.0 -0.0 0.029202 rpy=0.0 0.0 -0.011866 -> xyz=0.0 0.0 0.029202 rpy=0.0 0.0 -0.011866
- joint pr2/narrow_stereo_l_stereo_camera_frame_joint: origin xyz=0.0 0.0 0.0 rpy=0.0 0.0 0.0 -> xyz=-0.0 0.0 0.0 rpy=0.0 0.0 0.0
- joint pr2/narrow_stereo_l_stereo_camera_optical_frame_joint: origin xyz=0.0 0.0 0.0 rpy=-1.570796 0.0 -1.570796 -> xyz=-0.0 0.0 0.0 rpy=-1.570796 0.0 -1.570796
- joint pr2/narrow_stereo_optical_frame_joint: origin xyz=0.0 0.0 0.0 rpy=-1.570796 0.0 -1.570796 -> xyz=-0.0 0.0 0.0 rpy=-1.570796 0.0 -1.570796
- joint pr2/narrow_stereo_r_stereo_camera_frame_joint: origin xyz=0.0 -0.09 0.0 rpy=0.0 0.0 0.0 -> xyz=-0.0 -0.09 0.0 rpy=0.0 0.0 0.0
- joint pr2/projector_wg6802418_child_frame_joint: origin xyz=0.0 0.0 0.0 rpy=-0.0 -1.570796 0.0 -> xyz=0.0 0.0 0.0 rpy=0.0 -1.570796 0.0
- joint pr2/r_forearm_cam_optical_frame_joint: origin xyz=0.0 0.0 0.0 rpy=-1.570796 -0.0 -1.570796 -> xyz=0.0 0.0 0.0 rpy=-1.570796 0.0 -1.570796
- joint pr2/r_forearm_joint: origin xyz=-0.0 0.0 0.0 rpy=0.0 0.0 0.0 -> xyz=0.0 0.0 0.0 rpy=0.0 0.0 0.0
- joint pr2/r_gripper_tool_joint: origin xyz=0.18 0.0 -0.0 rpy=0.0 0.0 0.0 -> xyz=0.18 0.0 0.0 rpy=0.0 0.0 0.0
- joint pr2/t_torso_lift_side_item_profile_joint: origin xyz=0.0 0.0 0.52 rpy=1.570796 0.0 0.0 -> xyz=-0.0 0.0 0.52 rpy=1.570796 0.0 0.0
- joint pr2/wide_stereo_r_stereo_camera_optical_frame_joint: origin xyz=0.0 0.0 0.0 rpy=-1.570796 0.0 -1.570796 -> xyz=-0.0 0.0 0.0 rpy=-1.570796 0.0 -1.570796

Commit message: Name the slots the workflow sets vessels into in the location roles
A task names the poses it builds for the places of its layout
(RobotTaskDemo.named_places); a designator's pose that is one of them,
in the same frame at the same position and orientation, carries the
place's name in RoleSlot.place. The PR2 workflow names its rack,
refrigerator and centrifuge slots (rack A3, refrigerator R6, centrifuge
C4, ...), the recorded workflow carries them, and the Designators
panel shows them in all three panes.

Co-Authored-By: Claude Opus 5.5 <noreply@anthropic.com>

File: demo/standard_scenes/aicor_medical_lab_pr2_workflow/environment.urdf (robot description, URDF)
Before this commit: robot environment, 21 links, 20 joints
Links:
- removed link c83002c0-7c8c-45db-82c9-11bb0ee5c35a/odom
- added link 1f9635a1-2bab-4f59-9f08-1fa5e8687007/odom
Joints:
- removed joint c83002c0-7c8c-45db-82c9-11bb0ee5c35a/map_T_odom
- added joint 1f9635a1-2bab-4f59-9f08-1fa5e8687007/map_T_odom: type fixed, parent map, child 1f9635a1-2bab-4f59-9f08-1fa5e8687007/odom, origin xyz=0.0 0.0 0.0 rpy=0.0 0.0 0.0

File: demo/standard_scenes/aicor_medical_lab_pr2_workflow/pr2.urdf (robot description, URDF)
Before this commit: robot pr2, 105 links, 104 joints
Joints:
- joint pr2/l_force_torque_adapter_joint: origin xyz=0.0356 -0.0 0.0 rpy=0.0 -1.570796 0.0 -> xyz=0.0356 0.0 0.0 rpy=0.0 -1.570796 0.0
- joint pr2/l_forearm_cam_optical_frame_joint: origin xyz=-0.0 0.0 0.0 rpy=-1.570796 0.0 -1.570796 -> xyz=0.0 0.0 0.0 rpy=-1.570796 0.0 -1.570796
- joint pr2/l_forearm_joint: origin xyz=0.0 0.0 0.0 rpy=0.0 0.0 0.0 -> xyz=0.0 -0.0 0.0 rpy=0.0 0.0 0.0
- joint pr2/l_gripper_palm_joint: origin xyz=0.0 -0.0 0.0 rpy=1.22173 1.570796 0.0 -> xyz=0.0 0.0 0.0 rpy=1.22173 1.570796 0.0
- joint pr2/r_forearm_cam_optical_frame_joint: origin xyz=0.0 0.0 0.0 rpy=-1.570796 0.0 -1.570796 -> xyz=0.0 -0.0 0.0 rpy=-1.570796 0.0 -1.570796
- joint pr2/r_gripper_motor_accelerometer_joint: origin xyz=0.0 0.0 0.0 rpy=0.0 0.0 0.0 -> xyz=-0.0 0.0 0.0 rpy=0.0 0.0 0.0
- joint pr2/r_gripper_palm_joint: origin xyz=0.0 0.0 0.0 rpy=0.0 0.0 0.0 -> xyz=-0.0 0.0 0.0 rpy=0.0 0.0 0.0
- joint pr2/r_gripper_tool_joint: origin xyz=0.18 0.0 0.0 rpy=0.0 0.0 0.0 -> xyz=0.18 0.0 -0.0 rpy=0.0 0.0 0.0
- joint pr2/wide_stereo_r_stereo_camera_optical_frame_joint: origin xyz=-0.0 0.0 0.0 rpy=-1.570796 0.0 -1.570796 -> xyz=0.0 0.0 0.0 rpy=-1.570796 0.0 -1.570796
