Commit message: Record the frames each motion runs in
Every recorded frame names the motion coraplex reports running
(RecordedFrame.motion_node), and the frames each plan node ran in are
read from it as well as from the deepest running action: a motion, and
the sequence holding it, get frames of their own, and an action ends
with its last motion. The Designators panel shows each motion's own
phase and marks the running motion as current; a node that ran but
whose status coraplex never set, such as a sequence, shows as ended.
Both PR2 laboratory bundles are recorded again; every motion of the
workflow has frames, and the measurements are unchanged.

Co-Authored-By: Claude Opus 5.5 <noreply@anthropic.com>

File: demo/standard_scenes/aicor_medical_lab_pr2_query_stepper/environment.urdf (robot description, URDF)
Before this commit: robot environment, 21 links, 20 joints
Links:
- removed link 7f1cc62a-140a-4bcb-bad1-60de8f61831c/odom
- added link f1a8be4e-bc86-410a-a9cc-f184cfbd99dd/odom
Joints:
- removed joint 7f1cc62a-140a-4bcb-bad1-60de8f61831c/map_T_odom
- added joint f1a8be4e-bc86-410a-a9cc-f184cfbd99dd/map_T_odom: type fixed, parent map, child f1a8be4e-bc86-410a-a9cc-f184cfbd99dd/odom, origin xyz=0.0 0.0 0.0 rpy=0.0 0.0 0.0

File: demo/standard_scenes/aicor_medical_lab_pr2_workflow/environment.urdf (robot description, URDF)
Before this commit: robot environment, 21 links, 20 joints
Links:
- removed link 51529858-a0e4-46a0-b4f0-793ef5a077ab/odom
- added link 0b915927-c343-4893-93f8-f57fe1b447b8/odom
Joints:
- removed joint 51529858-a0e4-46a0-b4f0-793ef5a077ab/map_T_odom
- added joint 0b915927-c343-4893-93f8-f57fe1b447b8/map_T_odom: type fixed, parent map, child 0b915927-c343-4893-93f8-f57fe1b447b8/odom, origin xyz=0.0 0.0 0.0 rpy=0.0 0.0 0.0

File: demo/standard_scenes/aicor_medical_lab_pr2_workflow/pr2.urdf (robot description, URDF)
Before this commit: robot pr2, 105 links, 104 joints
Joints:
- joint pr2/l_force_torque_adapter_joint: origin xyz=0.0356 0.0 0.0 rpy=0.0 -1.570796 0.0 -> xyz=0.0356 -0.0 0.0 rpy=0.0 -1.570796 0.0
- joint pr2/l_forearm_cam_optical_frame_joint: origin xyz=0.0 0.0 0.0 rpy=-1.570796 0.0 -1.570796 -> xyz=-0.0 0.0 -0.0 rpy=-1.570796 0.0 -1.570796
- joint pr2/l_forearm_joint: origin xyz=0.0 -0.0 0.0 rpy=0.0 0.0 0.0 -> xyz=0.0 0.0 0.0 rpy=0.0 0.0 0.0
- joint pr2/narrow_stereo_r_stereo_camera_frame_joint: origin xyz=-0.0 -0.09 0.0 rpy=0.0 0.0 0.0 -> xyz=-0.0 -0.09 -0.0 rpy=0.0 0.0 0.0
- joint pr2/r_forearm_cam_optical_frame_joint: origin xyz=0.0 0.0 0.0 rpy=-1.570796 0.0 -1.570796 -> xyz=0.0 0.0 0.0 rpy=-1.570796 -0.0 -1.570796
- joint pr2/r_forearm_joint: origin xyz=0.0 -0.0 0.0 rpy=0.0 0.0 0.0 -> xyz=0.0 0.0 0.0 rpy=0.0 0.0 0.0
- joint pr2/wide_stereo_r_stereo_camera_frame_joint: origin xyz=0.0 -0.09 0.0 rpy=0.0 0.0 0.0 -> xyz=-0.0 -0.09 0.0 rpy=0.0 0.0 0.0
- joint pr2/wide_stereo_r_stereo_camera_optical_frame_joint: origin xyz=0.0 0.0 0.0 rpy=-1.570796 0.0 -1.570796 -> xyz=-0.0 0.0 0.0 rpy=-1.570796 0.0 -1.570796

Commit message: Mark the running step's target in the 3D view
Role slots record a pose's position and orientation in the frame of its
reference body (RoleSlot.pose). The Designators panel publishes where
the running step acts (ViewerEvent.TARGET_MARKED): the motion's
location, else its action's, else the entity it acts on; TargetMarker
attaches a mark to that body at the pose, so it moves with the body and
is drawn over what hides it, and highlights of the body leave it out.
At the end of the lowering into centrifuge C4 the gripper's tool frame
sits on the mark. Both PR2 laboratory bundles are recorded again with
the poses.

Co-Authored-By: Claude Opus 5.5 <noreply@anthropic.com>

File: demo/standard_scenes/aicor_medical_lab_pr2_query_stepper/environment.urdf (robot description, URDF)
Before this commit: robot environment, 21 links, 20 joints
Links:
- removed link f1a8be4e-bc86-410a-a9cc-f184cfbd99dd/odom
- added link a6409c87-9f78-4728-8641-8b8f964ae078/odom
Joints:
- removed joint f1a8be4e-bc86-410a-a9cc-f184cfbd99dd/map_T_odom
- added joint a6409c87-9f78-4728-8641-8b8f964ae078/map_T_odom: type fixed, parent map, child a6409c87-9f78-4728-8641-8b8f964ae078/odom, origin xyz=0.0 0.0 0.0 rpy=0.0 0.0 0.0

File: demo/standard_scenes/aicor_medical_lab_pr2_workflow/environment.urdf (robot description, URDF)
Before this commit: robot environment, 21 links, 20 joints
Links:
- removed link 0b915927-c343-4893-93f8-f57fe1b447b8/odom
- added link 301e0ace-1b2f-4c54-9599-2841ba8b4697/odom
Joints:
- removed joint 0b915927-c343-4893-93f8-f57fe1b447b8/map_T_odom
- added joint 301e0ace-1b2f-4c54-9599-2841ba8b4697/map_T_odom: type fixed, parent map, child 301e0ace-1b2f-4c54-9599-2841ba8b4697/odom, origin xyz=0.0 0.0 0.0 rpy=0.0 0.0 0.0

File: demo/standard_scenes/aicor_medical_lab_pr2_workflow/pr2.urdf (robot description, URDF)
Before this commit: robot pr2, 105 links, 104 joints
Joints:
- joint pr2/l_forearm_cam_optical_frame_joint: origin xyz=-0.0 0.0 -0.0 rpy=-1.570796 0.0 -1.570796 -> xyz=0.0 0.0 0.0 rpy=-1.570796 0.0 -1.570796
- joint pr2/l_forearm_joint: origin xyz=0.0 0.0 0.0 rpy=0.0 0.0 0.0 -> xyz=-0.0 -0.0 0.0 rpy=0.0 0.0 0.0
- joint pr2/l_gripper_tool_joint: origin xyz=0.18 -0.0 0.0 rpy=0.0 0.0 0.0 -> xyz=0.18 0.0 0.0 rpy=0.0 0.0 0.0
- joint pr2/l_upper_arm_joint: origin xyz=0.0 0.0 0.0 rpy=0.0 0.0 0.0 -> xyz=0.0 0.0 -0.0 rpy=0.0 0.0 0.0
- joint pr2/narrow_stereo_r_stereo_camera_frame_joint: origin xyz=-0.0 -0.09 -0.0 rpy=0.0 0.0 0.0 -> xyz=-0.0 -0.09 0.0 rpy=0.0 0.0 0.0
- joint pr2/r_forearm_cam_optical_frame_joint: origin xyz=0.0 0.0 0.0 rpy=-1.570796 -0.0 -1.570796 -> xyz=0.0 0.0 0.0 rpy=-1.570796 0.0 -1.570796
- joint pr2/r_gripper_led_joint: origin xyz=0.0513 0.0 0.0244 rpy=0.0 0.0 0.0 -> xyz=0.0513 -0.0 0.0244 rpy=0.0 0.0 0.0
- joint pr2/r_gripper_motor_accelerometer_joint: origin xyz=0.0 0.0 0.0 rpy=0.0 0.0 0.0 -> xyz=0.0 -0.0 0.0 rpy=0.0 0.0 0.0
- joint pr2/r_gripper_palm_joint: origin xyz=0.0 0.0 0.0 rpy=0.0 0.0 0.0 -> xyz=0.0 -0.0 0.0 rpy=0.0 0.0 0.0
- joint pr2/r_gripper_tool_joint: origin xyz=0.18 0.0 0.0 rpy=0.0 0.0 0.0 -> xyz=0.18 -0.0 0.0 rpy=0.0 0.0 0.0
- joint pr2/r_upper_arm_joint: origin xyz=0.0 0.0 0.0 rpy=0.0 0.0 0.0 -> xyz=0.0 -0.0 0.0 rpy=0.0 0.0 0.0
- joint pr2/wide_stereo_r_stereo_camera_frame_joint: origin xyz=-0.0 -0.09 0.0 rpy=0.0 0.0 0.0 -> xyz=0.0 -0.09 0.0 rpy=0.0 0.0 0.0
- joint pr2/wide_stereo_r_stereo_camera_optical_frame_joint: origin xyz=-0.0 0.0 0.0 rpy=-1.570796 0.0 -1.570796 -> xyz=0.0 0.0 0.0 rpy=-1.570796 0.0 -1.570796
